File: motorcontoller/KiCad/motorcontrol/motorcontrol.kicad_sch (KiCad schematic)
At the start: 77 parts, among them IC1 1EDN7126GXTMA1, IC10 1EDN7126GXTMA1, IC11 TMP236AQDBZTQ1, IC12 TLI4971A075T5UE0001XUMA1, IC13 TMUX6211RUMR, IC2 1EDN7126GXTMA1, IC3 TMP236AQDBZTQ1, IC4 TLI4971A075T5UE0001XUMA1, IC5 1EDN7126GXTMA1, IC6 1EDN7126GXTMA1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

Commit message: update
Parts:
- removed IC13: TMUX6211RUMR, QFN65P400X400X80-17N-D, symbol SamacSys_Parts:TMUX6211RUMR
- added C32: 6.8 nF, symbol Device:C_Small
- added IC13: SN74HC4851DGVR, SOP40P640X120-16N, symbol SamacSys_Parts:SN74HC4851DGVR
- added R22, R23, R24, R25, R26, R27, R28, R29: R, symbol Device:R_Small
- C17, C27, C3: value C -> 1 nF
- C19, C4: value 0.1 uF -> 6.8 nF
- C20, C30, C5: value C -> 226.8 nF
- R1, R13, R14, R20, R21, R3: value R -> 1 k
- R12, R19, R2: value R -> 4.7 k
Connections:
- net A1: now also IC13.3 (COM); no longer IC3.2 (VOUT)
- net A2_1: now also R24.2
- net A3_1: now also R25.2
- net A4_1: now also R26.2
- net A5_1: now also R29.2
- net D12: now also IC13.10 (B)
- net D13: now also IC13.9 (C)
- net D8: now also IC13.11 (A)
- net GND: now also C32.1, IC13.6 (INH), IC13.8 (GND)
- net V5: now also IC13.16 (VCC); no longer C4.2
- net A3: now reaches A2.A3
- net A1_I: now reaches IC4.4 (AOUT)
- net A1_I: now also C32.2, R23.2
- net A3_I: now reaches C19.2
- net A3_I: now also IC12.4 (AOUT), R28.2
- net A2_I: now reaches IC8.4 (AOUT)
- net A2_I: now also C4.2, R27.2
- net D1: no longer names the net of A2.D1 (D1/TX)
- new net: IC13.1 (Y4), R26.1
- new net: IC13.12 (Y3), R25.1
- new net: IC13.13 (Y0), R22.1
- new net: IC13.14 (Y1), R23.1
- new net: IC13.15 (Y2), R24.1
- new net: IC13.2 (Y6), R27.1
- new net: IC13.4 (Y7), R28.1
- new net: IC13.5 (Y5), R29.1
- new net A1_1: IC3.2 (VOUT), R22.2
