File: motorcontoller/KiCad/motorcontrol/motorcontrol.kicad_sch (KiCad schematic)
At the start: 86 parts, among them IC1 1EDN7126GXTMA1, IC10 1EDN7126GXTMA1, IC11 TMP236AQDBZTQ1, IC12 TLI4971A075T5UE0001XUMA1, IC13 SN74HC4851DGVR, IC2 1EDN7126GXTMA1, IC3 TMP236AQDBZTQ1, IC4 TLI4971A075T5UE0001XUMA1, IC5 1EDN7126GXTMA1, IC6 1EDN7126GXTMA1, IC7 TMP236AQDBZTQ1, IC8 TLI4971A075T5UE0001XUMA1, IC9 1EDN7126GXTMA1, J1 Screw_Terminal_For_Brushless_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, Q1 IGT60R070D1, Q2 IGT60R070D1, Q3 IGT60R070D1, Q4 IGT60R070D1, Q5 IGT60R070D1, Q6 IGT60R070D1, U1 AS5048B

Commit message: update
Parts:
- D?: renamed from D3; value 1N4001 -> 1N4007; symbol Diode:1N4001 -> Diode:1N4007
- D?: renamed from D1; value 1N4001 -> 1N4007; symbol Diode:1N4001 -> Diode:1N4007
- D?: renamed from D2; value 1N4001 -> 1N4007; symbol Diode:1N4001 -> Diode:1N4007
- IC1, IC2: footprint 1EDN7126GXTMA1 -> SamacSys_Parts:1EDN7126GXTMA1
- IC10: renamed from IC9; footprint 1EDN7126GXTMA1 -> SamacSys_Parts:1EDN7126GXTMA1
- IC11: renamed from IC10; footprint 1EDN7126GXTMA1 -> SamacSys_Parts:1EDN7126GXTMA1
- IC12: renamed from IC11; footprint SOT95P237X112-3N -> SamacSys_Parts:SOT95P237X112-3N
- IC13: renamed from IC12; footprint TLI4971A075T5UE0001XUMA1 -> SamacSys_Parts:TLI4971A075T5UE0001XUMA1
- IC3: footprint SOT95P237X112-3N -> SamacSys_Parts:SOT95P237X112-3N
- IC4: footprint TLI4971A075T5UE0001XUMA1 -> SamacSys_Parts:TLI4971A075T5UE0001XUMA1
- IC5: renamed from IC13; footprint SOP40P640X120-16N -> SamacSys_Parts:SOP40P640X120-16N
- IC6: renamed from IC5; footprint 1EDN7126GXTMA1 -> SamacSys_Parts:1EDN7126GXTMA1
- IC7: renamed from IC6; footprint 1EDN7126GXTMA1 -> SamacSys_Parts:1EDN7126GXTMA1
- IC8: renamed from IC7; footprint SOT95P237X112-3N -> SamacSys_Parts:SOT95P237X112-3N
- IC9: renamed from IC8; footprint TLI4971A075T5UE0001XUMA1 -> SamacSys_Parts:TLI4971A075T5UE0001XUMA1
- renumbered A2 to A1, C7 to C1, C5 to C10, C31 to C15, C15 to C16, C16 to C17, C29 to C18, C17 to C19, C8 to C2, C18 to C20, C4 to C21, C20 to C22, C21 to C23, C22 to C24, C23 to C25, C24 to C26, C25 to C27, C26 to C28, C27 to C29, C1 to C3, C28 to C30, C19 to C31, C30 to C32, C2 to C4, C9 to C5, C10 to C6, C3 to C7, C6 to C8, C32 to C9, R4 to R1, R28 to R10, R29 to R11, R8 to R12, R9 to R13, R24 to R14, R23 to R15, R22 to R16, R25 to R17, R10 to R18, R11 to R19, R6 to R2, R12 to R20, R13 to R21, R14 to R22, R15 to R23, R16 to R24, R17 to R25, R18 to R26, R19 to R27, R20 to R28, R21 to R29, R5 to R3, R7 to R4, R2 to R5, R1 to R6, R3 to R7, R26 to R8, R27 to R9
